File: Stackduino-SMD.sch (EAGLE design)
At the start: 55 parts, among them IC1 MCP23017SS, IC2 LM2675M, IC3 A3967SLB, SW1 ROTARTY_ENCODER, U2 ATMEGA328P, U3 FT232RLSSOP, U4 LTC2950CTS8-1TRPBF, U5 LTC4412ES6PBF, Y1 16MHz

Commit message: latest progress
Parts:
- removed OK2: 4N35SM, optocoupler:4N35SM
- added OK3: LTV816S, optocoupler:LTV816S
- added R22: 470K, SparkFun-Resistors:1KOHM1/10W1%(0603)
- OK1: value 4N35SM -> LTV816S; device optocoupler:4N35SM -> optocoupler:LTV816S
- S2: value (none) -> Start/Stop
- S3: value (none) -> Forward
- S4: value (none) -> Backward
Connections:
- new net STAT: IC1.GPA4, R22.1, U5.STAT
- net +5V: now also R22.2
- net GND: no longer OK1.C, OK1.EMI, OK2.C, OK2.EMI
- net N$36: now also OK3.A; no longer OK2.A
- net OPT1: no longer OK1.COL
- net OPT2: no longer OK2.COL
Changed lines of the file:
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@@
 <part name="SW1" library="SparkFun-Electromechanical" deviceset="ROTARTY_ENCODER" device=""/>
 <part name="S1" library="SparkFun-Electromechanical" deviceset="TAC_SWITCH" device="PTH"/>
-<part name="S2" library="SparkFun-Electromechanical" deviceset="TAC_SWITCH" device="PTH"/>
+<part name="S2" library="SparkFun-Electromechanical" deviceset="TAC_SWITCH" device="PTH" value="Start/Stop"/>
 <part name="U$2" library="Stackduino" deviceset="DIGOLE_OLED" device=""/>
 <part name="U3" library="SparkFun-DigitalIC" deviceset="FT232RL" device="SSOP"/>
@@
 <part name="SUPPLY21" library="supply2" deviceset="GND" device=""/>
 <part name="SUPPLY23" library="supply2" deviceset="GND" device=""/>
-<part name="S3" library="SparkFun-Electromechanical" deviceset="TAC_SWITCH" device="PTH"/>
-<part name="S4" library="SparkFun-Electromechanical" deviceset="TAC_SWITCH" device="PTH"/>
+<part name="S3" library="SparkFun-Electromechanical" deviceset="TAC_SWITCH" device="PTH" value="Forward"/>
+<part name="S4" library="SparkFun-Electromechanical" deviceset="TAC_SWITCH" device="PTH" value="Backward"/>
 <part name="JP2" library="avr-5" deviceset="AVR-ISP-6" device=""/>
 <part name="SUPPLY24" library="supply2" deviceset="GND" device=""/>
@@
 <part name="SUPPLY27" library="supply2" deviceset="GND" device=""/>
 <part name="SUPPLY28" library="supply2" deviceset="GND" device=""/>
-<part name="OK1" library="optocoupler" deviceset="4N*?M" device="S" technology="35"/>
-<part name="OK2" library="optocoupler" deviceset="4N*?M" device="S" technology="35"/>
 <part name="SUPPLY29" library="supply2" deviceset="GND" device=""/>
 <part name="SUPPLY30" library="supply2" deviceset="GND" device=""/>
@@
 <part name="C8" library="SparkFun-Capacitors" deviceset="CAP_POL" device="G" value="47uF"/>
 <part name="GND1" library="supply2" deviceset="GND" device=""/>
+<part name="P+19" library="supply1" deviceset="+5V" device="" value="VCC"/>
+<part name="R22" library="SparkFun-Resistors" deviceset="1KOHM1/10W1%(0603)" device="" value="470K"/>
+<part name="OK3" library="optocoupler" deviceset="LTV816" device="S"/>
+<part name="OK1" library="optocoupler" deviceset="LTV816" device="S"/>
 </parts>
 <sheets>
@@
 <instance part="SUPPLY27" gate="GND" x="15.24" y="25.4"/>
 <instance part="SUPPLY28" gate="GND" x="-22.86" y="30.48"/>
-<instance part="OK1" gate="G$1" x="78.74" y="38.1"/>
-<instance part="OK2" gate="G$1" x="78.74" y="17.78"/>
-<instance part="SUPPLY29" gate="GND" x="58.42" y="10.16"/>
-<instance part="SUPPLY30" gate="GND" x="58.42" y="30.48"/>
-<instance part="SUPPLY31" gate="GND" x="96.52" y="10.16"/>
-<instance part="SUPPLY32" gate="GND" x="96.52" y="30.48"/>
+<instance part="SUPPLY29" gate="GND" x="58.42" y="12.7"/>
+<instance part="SUPPLY30" gate="GND" x="58.42" y="33.02"/>
+<instance part="SUPPLY31" gate="GND" x="96.52" y="12.7"/>
+<instance part="SUPPLY32" gate="GND" x="96.52" y="33.02"/>
 <instance part="SUPPLY33" gate="GND" x="-218.44" y="-93.98"/>
 <instance part="SUPPLY34" gate="GND" x="-218.44" y="-78.74"/>
@@
 <instance part="C8" gate="G$1" x="109.22" y="116.84" rot="R180"/>
 <instance part="GND1" gate="GND" x="109.22" y="104.14"/>
+<instance part="P+19" gate="1" x="-152.4" y="88.9" smashed="yes">
+<attribute name="VALUE" x="-150.114" y="87.122" size="1.778" layer="96"/>
+</instance>
+<instance part="R22" gate="G$1" x="-152.4" y="78.74" rot="R90"/>
+<instance part="OK3" gate="G$1" x="78.74" y="17.78"/>
+<instance part="OK1" gate="G$1" x="78.74" y="38.1"/>
 </instances>
 <busses>
@@
 </segment>
 <segment>
-<pinref part="OK1" gate="G$1" pin="C"/>
 <pinref part="SUPPLY30" gate="GND" pin="GND"/>
-<wire x1="68.58" y1="33.02" x2="58.42" y2="33.02" width="0.1524" layer="91"/>
-</segment>
-<segment>
-<pinref part="OK2" gate="G$1" pin="C"/>
+<wire x1="68.58" y1="35.56" x2="58.42" y2="35.56" width="0.1524" layer="91"/>
+</segment>
+<segment>
 <pinref part="SUPPLY29" gate="GND" pin="GND"/>
-<wire x1="68.58" y1="12.7" x2="58.42" y2="12.7" width="0.1524" layer="91"/>
-</segment>
-<segment>
-<pinref part="OK1" gate="G$1" pin="EMI"/>
+<wire x1="68.58" y1="15.24" x2="58.42" y2="15.24" width="0.1524" layer="91"/>
+</segment>
+<segment>
 <pinref part="SUPPLY32" gate="GND" pin="GND"/>
-<wire x1="86.36" y1="33.02" x2="96.52" y2="33.02" width="0.1524" layer="91"/>
-</segment>
-<segment>
-<pinref part="OK2" gate="G$1" pin="EMI"/>
+<wire x1="86.36" y1="35.56" x2="96.52" y2="35.56" width="0.1524" layer="91"/>
+</segment>
+<segment>
 <pinref part="SUPPLY31" gate="GND" pin="GND"/>
-<wire x1="86.36" y1="12.7" x2="96.52" y2="12.7" width="0.1524" layer="91"/>
+<wire x1="86.36" y1="15.24" x2="96.52" y2="15.24" width="0.1524" layer="91"/>
 </segment>
 <segment>
@@
 </segment>
 <segment>
-<wire x1="-187.96" y1="45.72" x2="-187.96" y2="45.974" width="0.1524" layer="91"/>
 <wire x1="-187.96" y1="45.974" x2="-187.96" y2="48.26" width="0.1524" layer="91"/>
 <wire x1="-187.96" y1="48.26" x2="-172.72" y2="48.26" width="0.1524" layer="91"/>
@@
 <wire x1="-172.72" y1="48.26" x2="-172.72" y2="30.48" width="0.1524" layer="91"/>
 <pinref part="U$1" gate="G$1" pin="10"/>
-<junction x="-187.96" y="45.974"/>
 </segment>
 <segment>
@@
 <pinref part="GND1" gate="GND" pin="GND"/>
 </segment>
-</net>
-<net name="N$9" class="0">
 <segment>
 <wire x1="-5.08" y1="101.6" x2="-5.08" y2="104.14" width="0.1524" layer="91"/>
@@
 <wire x1="-111.76" y1="15.24" x2="-111.76" y2="43.18" width="0.1524" layer="91"/>
 <pinref part="P+18" gate="1" pin="+5V"/>
+</segment>
+<segment>
+<pinref part="P+19" gate="1" pin="+5V"/>
+<pinref part="R22" gate="G$1" pin="2"/>
+<wire x1="-152.4" y1="86.36" x2="-152.4" y2="83.82" width="0.1524" layer="91"/>
 </segment>
 </net>
@@
 <net name="OPT1" class="0">
 <segment>
-<pinref part="OK1" gate="G$1" pin="COL"/>
-<wire x1="86.36" y1="38.1" x2="96.52" y2="38.1" width="0.1524" layer="91"/>
+<wire x1="86.36" y1="40.64" x2="96.52" y2="40.64" width="0.1524" layer="91"/>
 <label x="99.06" y="38.1" size="1.778" layer="95"/>
 </segment>
@@
 <label x="-195.58" y="76.2" size="1.778" layer="95"/>
 <pinref part="U$1" gate="G$1" pin="8"/>
-<junction x="-198.12" y="45.974"/>
 </segment>
 </net>
 <net name="OPT2" class="0">
 <segment>
-<pinref part="OK2" gate="G$1" pin="COL"/>
-<wire x1="86.36" y1="17.78" x2="96.52" y2="17.78" width="0.1524" layer="91"/>
+<wire x1="86.36" y1="20.32" x2="96.52" y2="20.32" width="0.1524" layer="91"/>
 <label x="99.06" y="17.78" size="1.778" layer="95"/>
 </segment>
@@
 <label x="-187.96" y="83.82" size="1.778" layer="95"/>
 <pinref part="U$1" gate="G$1" pin="9"/>
-<junction x="-193.04" y="45.974"/>
 </segment>
 </net>
@@
 <pinref part="U$1" gate="G$1" pin="6"/>
 <wire x1="-208.28" y1="45.974" x2="-208.28" y2="73.66" width="0.1524" layer="91"/>
-<junction x="-208.28" y="45.974"/>
 </segment>
 </net>
@@
 <pinref part="U$1" gate="G$1" pin="7"/>
 <wire x1="-203.2" y1="45.974" x2="-203.2" y2="66.04" width="0.1524" layer="91"/>
-<junction x="-203.2" y="45.974"/>
 </segment>
 </net>
 <net name="LIM1" class="0">
 <segment>
-<wire x1="-205.74" y1="45.72" x2="-205.74" y2="45.974" width="0.1524" layer="91"/>
 <wire x1="-205.74" y1="45.974" x2="-205.74" y2="58.42" width="0.1524" layer="91"/>
 <wire x1="-205.74" y1="58.42" x2="-185.42" y2="58.42" width="0.1524" layer="91"/>
@@
 <label x="-170.18" y="73.66" size="1.778" layer="95"/>
 <pinref part="U$1" gate="G$1" pin="11"/>
-<junction x="-205.74" y="45.974"/>
 </segment>
 <segment>
@@
 <label x="-170.18" y="63.5" size="1.778" layer="95"/>
 <pinref part="U$1" gate="G$1" pin="12"/>
-<junction x="-200.66" y="45.974"/>
 </segment>
 <segment>
@@
 <label x="-170.18" y="55.88" size="1.778" layer="95"/>
 <pinref part="U$1" gate="G$1" pin="13"/>
-<junction x="-195.58" y="45.974"/>
 </segment>
 <segment>
@@
 <net name="DIG2" class="0">
 <segment>
-<wire x1="-190.5" y1="45.72" x2="-190.5" y2="45.974" width="0.1524" layer="91"/>
 <wire x1="-190.5" y1="45.974" x2="-190.5" y2="50.8" width="0.1524" layer="91"/>
 <wire x1="-190.5" y1="50.8" x2="-172.72" y2="50.8" width="0.1524" layer="91"/>
 <label x="-170.18" y="50.8" size="1.778" layer="95"/>
 <pinref part="U$1" gate="G$1" pin="14"/>
-<junction x="-190.5" y="45.974"/>
 </segment>
 <segment>
@@
 <wire x1="-160.02" y1="-53.34" x2="-198.12" y2="-53.34" width="0.1524" layer="91"/>
 <label x="190.5" y="76.2" size="1.778" layer="95"/>
+<label x="-215.9" y="-53.34" size="1.778" layer="95"/>
 </segment>
 <segment>
@@
 <segment>
 <pinref part="R3" gate="G$1" pin="1"/>
+<wire x1="55.88" y1="40.64" x2="68.58" y2="40.64" width="0.1524" layer="91"/>
 <pinref part="OK1" gate="G$1" pin="A"/>
-<wire x1="55.88" y1="40.64" x2="68.58" y2="40.64" width="0.1524" layer="91"/>
 </segment>
 </net>
@@
 <segment>
 <pinref part="R4" gate="G$1" pin="1"/>
-<pinref part="OK2" gate="G$1" pin="A"/>
 <wire x1="55.88" y1="20.32" x2="68.58" y2="20.32" width="0.1524" layer="91"/>
+<pinref part="OK3" gate="G$1" pin="A"/>
 </segment>
 </net>
@@
 </segment>
 </net>
+<net name="STAT" class="0">
+<segment>
+<pinref part="R22" gate="G$1" pin="1"/>
+<pinref part="U5" gate="A" pin="STAT"/>
+<wire x1="-152.4" y1="73.66" x2="-144.78" y2="73.66" width="0.1524" layer="91"/>
+<wire x1="-152.4" y1="73.66" x2="-152.4" y2="63.5" width="0.1524" layer="91"/>
+<junction x="-152.4" y="73.66"/>
+<label x="-149.86" y="63.5" size="1.778" layer="95"/>
+</segment>
+<segment>
+<pinref part="IC1" gate="G$1" pin="GPA4"/>
+<wire x1="-106.68" y1="-71.12" x2="-170.18" y2="-71.12" width="0.1524" layer="91"/>
+<wire x1="-170.18" y1="-71.12" x2="-170.18" y2="-58.42" width="0.1524" layer="91"/>
+<wire x1="-170.18" y1="-58.42" x2="-198.12" y2="-58.42" width="0.1524" layer="91"/>
+<label x="-205.74" y="-58.42" size="1.778" layer="95"/>
+</segment>
+</net>

Commit message: latest progress
Parts:
- removed C8: 47uF, SparkFun-Capacitors:CAP_POLG
- added C9: (no value), SparkFun-Passives:CAP_POLD
- CN1: value (none) -> Battery Connector
- S1: value (none) -> Start/Stop
- U$2: value (none) -> OLED Display
Connections:
- net N$12 renamed VDD
- net +5V: now also R19.2; no longer R19.1
- net GND: now also C9.-, OK1.C, OK1.EMIT, OK3.C, OK3.EMIT, U$1.15; no longer C8.+
- net N$18: now also R19.1; no longer R19.2
- net N$32: now also R4.2
- net OPT1: now also OK1.COL
- net OPT2: now also OK3.COL
- net V+: now also C9.+; no longer C8.-
Other:
- moved on the sheet: R19, U$1

Commit message: Initial layout of board
Parts:
- removed S1: Start/Stop, SparkFun-Electromechanical:TAC_SWITCHPTH
- added C10, C11, C8: 0.1uF, SparkFun-Capacitors:0.1UF-25V(+80/-20%)(0603)
- added S5: (no value), adafruit:40-XX-ROUND
- S2: value Start/Stop -> (none); device SparkFun-Electromechanical:TAC_SWITCHPTH -> adafruit:31-XX
- renumbered IC1 to MCP23017, IC2 to LM2675, IC3 to A3967, U2 to ATMEGA, U3 to FT232RL, U4 to LTC2950, U5 to LTC4412
Connections:
- net +5V: now also C10.2, C11.2, MCP23017.!RESET, MCP23017.VDD
- net GND: now also C10.1, C11.1, C8.2, S2.P, S5.S1; no longer S1.2, S2.4
- net N$28: now also S5.P1; no longer S2.2
- net N$8: now also S2.S; no longer S1.4
- net VCC: now also C8.1; no longer MCP23017.!RESET, MCP23017.VDD

Commit message: Substituted in a4988 polulu driver
Parts:
- removed A3967: A3967SLB, Allegro:A3967SLB
- removed C6: 680pF, SparkFun03_30_09:CAP0402
- removed R10, R11, R12, R13, R14, R15: 10K, SparkFun03_30_09:RESISTOR0402
- removed R16: TRIMPOTSMD, SparkFun:TRIMPOTSMD
- removed R17: ???, SparkFun03_30_09:RESISTOR0402
- removed R6: .75, rcl:R-US_R0805
- removed R7, R8: 20K, SparkFun03_30_09:RESISTOR0402
- removed R9: 5.1K, SparkFun03_30_09:RESISTOR0402
- removed TP1: TPPAD1-13, testpad:TPPAD1-13
- added U$3: A4988BREAKOUT, RepRapjr:A4988BREAKOUT
- C5: value 680pF -> 0.1uF; device SparkFun03_30_09:CAP0402 -> SparkFun-Capacitors:0.1UF-25V(+80/-20%)(0603)
- R5: value .75 -> 100K; device rcl:R-US_R0805 -> SparkFun-Resistors:1KOHM1/10W1%(0603)
Connections:
- removed net N$37: A3967.SENSE2, R5.2
- removed net N$38: A3967.SENSE1, R6.2
- removed net N$39: A3967.RC2, C5.1, R8.2
- removed net N$40: A3967.RC1, C6.1, R7.2
- removed net N$41: A3967.REF, R16.WIPER, TP1.TP
- removed net N$42: R16.CW, R9.2
- removed net PFD: A3967.PFD, R12.1, R17.2
- removed net RESET: A3967./RESET, R15.1
- new net MS3: MCP23017.GPB5, U$3.MS3
- new net N$2: R5.1, U$3.RST
- net +5V: now also C5.1, R5.2, U$3.VDD
- net DIR: now also U$3.DIR; no longer A3967.DIR
- net ENABLE: now also MCP23017.GPB6, U$3.EN; no longer A3967./ENABLE, MCP23017.GPB5, R13.2
- net GND: now also U$3.GND@0, U$3.GND@1; no longer A3967.GND1, A3967.GND2, A3967.GND3, A3967.GND4, C6.2, R13.1, R17.1, R5.1, R6.1, R7.1, R8.1, R9.1
- net MS1: now also U$3.MS1; no longer A3967.MS1, R14.1
- net MS2: now also U$3.MS2; no longer A3967.MS2, R10.1
- net OUT1A: now also U$3.1A; no longer A3967.OUT1A
- net OUT1B: now also U$3.1B; no longer A3967.OUT1B
- net OUT2A: now also U$3.2A; no longer A3967.OUT2A
- net OUT2B: now also U$3.2B; no longer A3967.OUT2B
- net SLEEP: now also MCP23017.GPB7, U$3.SLEEP; no longer A3967./SLEEP, MCP23017.GPB6, R11.1
- net STEP: now also U$3.STEP; no longer A3967.STEP
- net V+: now also U$3.VMOT; no longer A3967.LOAD_SUPPLY1, A3967.LOAD_SUPPLY2
- net VCC: no longer A3967.LOGIC_SUPPLY, R10.2, R11.2, R12.2, R14.2, R15.2, R16.CCW
Other:
- moved on the sheet: C5, R5

Commit message: Latest progress
Connections:
- net GND: now also 12VDC.RING_SW
Changed lines of the file:
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@@
 <grid distance="0.1" unitdist="inch" unit="inch" style="lines" multiple="1" display="no" altdistance="0.01" altunitdist="inch" altunit="inch"/>
 <layers>
-<layer number="1" name="Top" color="4" fill="1" visible="no" active="no"/>
-<layer number="16" name="Bottom" color="1" fill="1" visible="no" active="no"/>
-<layer number="17" name="Pads" color="2" fill="1" visible="no" active="no"/>
-<layer number="18" name="Vias" color="2" fill="1" visible="no" active="no"/>
-<layer number="19" name="Unrouted" color="6" fill="1" visible="no" active="no"/>
-<layer number="20" name="Dimension" color="15" fill="1" visible="no" active="no"/>
-<layer number="21" name="tPlace" color="7" fill="1" visible="no" active="no"/>
-<layer number="22" name="bPlace" color="7" fill="1" visible="no" active="no"/>
-<layer number="23" name="tOrigins" color="15" fill="1" visible="no" active="no"/>
-<layer number="24" name="bOrigins" color="15" fill="1" visible="no" active="no"/>
-<layer number="25" name="tNames" color="7" fill="1" visible="no" active="no"/>
-<layer number="26" name="bNames" color="7" fill="1" visible="no" active="no"/>
-<layer number="27" name="tValues" color="7" fill="1" visible="no" active="no"/>
-<layer number="28" name="bValues" color="7" fill="1" visible="no" active="no"/>
+<layer number="1" name="Top" color="4" fill="1" visible="yes" active="no"/>
+<layer number="16" name="Bottom" color="1" fill="1" visible="yes" active="no"/>
+<layer number="17" name="Pads" color="2" fill="1" visible="yes" active="no"/>
+<layer number="18" name="Vias" color="2" fill="1" visible="yes" active="no"/>
+<layer number="19" name="Unrouted" color="6" fill="1" visible="yes" active="no"/>
+<layer number="20" name="Dimension" color="15" fill="1" visible="yes" active="no"/>
+<layer number="21" name="tPlace" color="16" fill="1" visible="yes" active="no"/>
+<layer number="22" name="bPlace" color="14" fill="1" visible="yes" active="no"/>
+<layer number="23" name="tOrigins" color="15" fill="1" visible="yes" active="no"/>
+<layer number="24" name="bOrigins" color="15" fill="1" visible="yes" active="no"/>
+<layer number="25" name="tNames" color="7" fill="1" visible="yes" active="no"/>
+<layer number="26" name="bNames" color="7" fill="1" visible="yes" active="no"/>
+<layer number="27" name="tValues" color="7" fill="1" visible="yes" active="no"/>
+<layer number="28" name="bValues" color="7" fill="1" visible="yes" active="no"/>
 <layer number="29" name="tStop" color="7" fill="3" visible="no" active="no"/>
 <layer number="30" name="bStop" color="7" fill="6" visible="no" active="no"/>
@@
 <layer number="35" name="tGlue" color="7" fill="4" visible="no" active="no"/>
 <layer number="36" name="bGlue" color="7" fill="5" visible="no" active="no"/>
-<layer number="37" name="tTest" color="7" fill="1" visible="no" active="no"/>
-<layer number="38" name="bTest" color="7" fill="1" visible="no" active="no"/>
+<layer number="37" name="tTest" color="7" fill="1" visible="yes" active="no"/>
+<layer number="38" name="bTest" color="7" fill="1" visible="yes" active="no"/>
 <layer number="39" name="tKeepout" color="4" fill="11" visible="no" active="no"/>
 <layer number="40" name="bKeepout" color="1" fill="11" visible="no" active="no"/>
@@
 <layer number="44" name="Drills" color="7" fill="1" visible="no" active="no"/>
 <layer number="45" name="Holes" color="7" fill="1" visible="no" active="no"/>
-<layer number="46" name="Milling" color="3" fill="1" visible="no" active="no"/>
-<layer number="47" name="Measures" color="7" fill="1" visible="no" active="no"/>
-<layer number="48" name="Document" color="7" fill="1" visible="no" active="no"/>
-<layer number="49" name="Reference" color="7" fill="1" visible="no" active="no"/>
-<layer number="50" name="dxf" color="7" fill="1" visible="no" active="no"/>
-<layer number="51" name="tDocu" color="14" fill="1" visible="no" active="no"/>
-<layer number="52" name="bDocu" color="7" fill="1" visible="no" active="no"/>
-<layer number="53" name="tGND_GNDA" color="7" fill="9" visible="no" active="no"/>
-<layer number="54" name="bGND_GNDA" color="1" fill="9" visible="no" active="no"/>
-<layer number="56" name="wert" color="7" fill="1" visible="no" active="no"/>
-<layer number="57" name="tCAD" color="7" fill="1" visible="no" active="no"/>
+<layer number="46" name="Milling" color="3" fill="1" visible="yes" active="no"/>
+<layer number="47" name="Measures" color="7" fill="1" visible="yes" active="no"/>
+<layer number="48" name="Document" color="7" fill="1" visible="yes" active="no"/>
+<layer number="49" name="Reference" color="7" fill="1" visible="yes" active="no"/>
+<layer number="50" name="dxf" color="7" fill="1" visible="yes" active="no"/>
+<layer number="51" name="tDocu" color="6" fill="1" visible="yes" active="no"/>
+<layer number="52" name="bDocu" color="7" fill="1" visible="yes" active="no"/>
+<layer number="53" name="tGND_GNDA" color="7" fill="9" visible="yes" active="no"/>
+<layer number="54" name="bGND_GNDA" color="1" fill="9" visible="yes" active="no"/>
+<layer number="56" name="wert" color="7" fill="1" visible="yes" active="no"/>
+<layer number="57" name="tCAD" color="7" fill="1" visible="yes" active="no"/>
 <layer number="91" name="Nets" color="2" fill="1" visible="yes" active="yes"/>
 <layer number="92" name="Busses" color="1" fill="1" visible="yes" active="yes"/>
@@
 <pinref part="SUPPLY10" gate="GND" pin="GND"/>
 <wire x1="-149.86" y1="127" x2="-149.86" y2="129.54" width="0.1524" layer="91"/>
-</segment>
-<segment>
+<pinref part="12VDC" gate="G$1" pin="RING_SW"/>
+<wire x1="-149.86" y1="129.54" x2="-149.86" y2="132.08" width="0.1524" layer="91"/>
+<junction x="-149.86" y="129.54"/>
+</segment>
+<segment>

Commit message: Latest progress
Connections:
- removed net +5V: C10.2, C11.2, C5.1, FT232RL.VCC, FT232RL.VCCIO, JP2.2, MCP23017.!RESET, MCP23017.VDD, R18.1, R19.2, R22.2, R5.2, U$3.VDD
- net VCC: now also C10.2, C11.2, C5.1, FT232RL.VCC, FT232RL.VCCIO, JP2.2, MCP23017.!RESET, MCP23017.VDD, R18.1, R19.2, R22.2, R5.2, U$3.VDD

Commit message: Latest progress
Parts:
- CN1: device adafruit:JST_2PIN-SMT -> adafruit:JST_2PIN-THM
Changed lines of the file:
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@@
 <part name="SUPPLY14" library="supply2" deviceset="GND" device=""/>
 <part name="SUPPLY15" library="supply2" deviceset="GND" device=""/>
-<part name="CN1" library="adafruit" deviceset="JST_2PIN" device="-SMT" value="Battery Connector"/>
+<part name="CN1" library="adafruit" deviceset="JST_2PIN" device="-THM" value="Battery Connector"/>
 <part name="C4" library="SparkFun-Capacitors" deviceset="0.1UF-25V(+80/-20%)(0603)" device="" value="0.1uF"/>
 <part name="R1" library="SparkFun-Resistors" deviceset="1KOHM1/10W1%(0603)" device="" value="1.5K"/>
