File: Stackduino-SMD.sch (EAGLE design)
At the start: 45 parts, among them CN1 Battery Connector, SW1 ROTARTY_ENCODER, Y1 16MHz

Commit message: Latest progress
Parts:
- C10, C11, C4, C5, C7, C8: device SparkFun-Capacitors:0.1UF-25V(+80/-20%)(0603) -> eagle-ltspice:CC1206
- R1, R18, R19, R2, R20, R21, R3, R4: device SparkFun-Resistors:1KOHM1/10W1%(0603) -> rcl:R-EU_R1206
- R22: device SparkFun-Resistors:1KOHM1/10W1%(0603) -> eagle-ltspice:RR1206
- R5: device SparkFun-Resistors:1KOHM1/10W1%(0603) -> eagle-ltspice:CC1206
Other:
- moved on the sheet: C10, C11, C4, C5, C7
Changed lines of the file:
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@@
 <part name="SUPPLY15" library="supply2" deviceset="GND" device=""/>
 <part name="CN1" library="adafruit" deviceset="JST_2PIN" device="-THM" value="Battery Connector"/>
-<part name="C4" library="SparkFun-Capacitors" deviceset="0.1UF-25V(+80/-20%)(0603)" device="" value="0.1uF"/>
-<part name="R1" library="SparkFun-Resistors" deviceset="1KOHM1/10W1%(0603)" device="" value="1.5K"/>
+<part name="C4" library="eagle-ltspice" deviceset="C" device="C1206" value="0.1uF"/>
+<part name="R1" library="rcl" deviceset="R-EU_" device="R1206" value="1.5K"/>
 <part name="Y1" library="SparkFun-FreqCtrl" deviceset="RESONATOR" device="16MHZ" value="16MHz"/>
 <part name="SUPPLY19" library="supply2" deviceset="GND" device=""/>
@@
 <part name="SUPPLY36" library="supply2" deviceset="GND" device=""/>
 <part name="SUPPLY37" library="supply2" deviceset="GND" device=""/>
-<part name="R2" library="SparkFun-Resistors" deviceset="1KOHM1/10W1%(0603)" device="" value="10K"/>
-<part name="R3" library="SparkFun-Resistors" deviceset="1KOHM1/10W1%(0603)" device="" value="220K"/>
-<part name="R4" library="SparkFun-Resistors" deviceset="1KOHM1/10W1%(0603)" device="" value="220K"/>
+<part name="R2" library="rcl" deviceset="R-EU_" device="R1206" value="10K"/>
+<part name="R3" library="rcl" deviceset="R-EU_" device="R1206" value="220K"/>
+<part name="R4" library="rcl" deviceset="R-EU_" device="R1206" value="220K"/>
 <part name="P+2" library="supply1" deviceset="+5V" device="" value="VCC"/>
 <part name="P+4" library="supply1" deviceset="+5V" device="" value="VCC"/>
@@
 <part name="SUPPLY22" library="supply2" deviceset="GND" device=""/>
 <part name="P+14" library="supply1" deviceset="+5V" device="" value="VCC"/>
-<part name="R18" library="SparkFun-Resistors" deviceset="1KOHM1/10W1%(0603)" device="" value="4.7K"/>
+<part name="R18" library="rcl" deviceset="R-EU_" device="R1206" value="4.7K"/>
 <part name="P+18" library="supply1" deviceset="+5V" device="" value="VCC"/>
-<part name="R20" library="SparkFun-Resistors" deviceset="1KOHM1/10W1%(0603)" device="" value="4.7K"/>
-<part name="R21" library="SparkFun-Resistors" deviceset="1KOHM1/10W1%(0603)" device="" value="10K"/>
+<part name="R20" library="rcl" deviceset="R-EU_" device="R1206" value="4.7K"/>
+<part name="R21" library="rcl" deviceset="R-EU_" device="R1206" value="10K"/>
 <part name="SUPPLY25" library="supply2" deviceset="GND" device=""/>
-<part name="C7" library="SparkFun-Capacitors" deviceset="0.1UF-25V(+80/-20%)(0603)" device="" value="100nF"/>
+<part name="C7" library="eagle-ltspice" deviceset="C" device="C1206" value="100nF"/>
 <part name="SUPPLY38" library="supply2" deviceset="GND" device=""/>
 <part name="GND1" library="supply2" deviceset="GND" device=""/>
 <part name="P+19" library="supply1" deviceset="+5V" device="" value="VCC"/>
-<part name="R22" library="SparkFun-Resistors" deviceset="1KOHM1/10W1%(0603)" device="" value="470K"/>
+<part name="R22" library="eagle-ltspice" deviceset="R" device="R1206" value="470K"/>
 <part name="OK3" library="optocoupler" deviceset="LTV816" device="S"/>
 <part name="OK1" library="optocoupler" deviceset="LTV816" device="S"/>
-<part name="R19" library="SparkFun-Resistors" deviceset="1KOHM1/10W1%(0603)" device="" value="4.7K"/>
+<part name="R19" library="rcl" deviceset="R-EU_" device="R1206" value="4.7K"/>
 <part name="P+17" library="supply1" deviceset="+5V" device="" value="VCC"/>
 <part name="C9" library="SparkFun-Passives" deviceset="CAP_POL" device="D"/>
 <part name="S5" library="adafruit" deviceset="40-XX" device="-ROUND"/>
 <part name="S2" library="adafruit" deviceset="31-XX" device=""/>
-<part name="C8" library="SparkFun-Capacitors" deviceset="0.1UF-25V(+80/-20%)(0603)" device="" value="0.1uF"/>
+<part name="C8" library="eagle-ltspice" deviceset="C" device="C1206" value="0.1uF"/>
 <part name="SUPPLY39" library="supply2" deviceset="GND" device=""/>
-<part name="C10" library="SparkFun-Capacitors" deviceset="0.1UF-25V(+80/-20%)(0603)" device="" value="0.1uF"/>
+<part name="C10" library="eagle-ltspice" deviceset="C" device="C1206" value="0.1uF"/>
 <part name="GND2" library="supply2" deviceset="GND" device=""/>
-<part name="C11" library="SparkFun-Capacitors" deviceset="0.1UF-25V(+80/-20%)(0603)" device="" value="0.1uF"/>
+<part name="C11" library="eagle-ltspice" deviceset="C" device="C1206" value="0.1uF"/>
 <part name="GND3" library="supply2" deviceset="GND" device=""/>
 <part name="U$3" library="RepRapjr" deviceset="A4988BREAKOUT" device=""/>
@@
 <part name="P+20" library="supply1" deviceset="+5V" device="" value="VCC"/>
 <part name="SUPPLY41" library="supply2" deviceset="GND" device=""/>
-<part name="R5" library="SparkFun-Resistors" deviceset="1KOHM1/10W1%(0603)" device="" value="100K"/>
+<part name="R5" library="eagle-ltspice" deviceset="C" device="C1206" value="100K"/>
 <part name="P+1" library="supply1" deviceset="+5V" device="" value="VCC"/>
-<part name="C5" library="SparkFun-Capacitors" deviceset="0.1UF-25V(+80/-20%)(0603)" device="" value="0.1uF"/>
+<part name="C5" library="eagle-ltspice" deviceset="C" device="C1206" value="0.1uF"/>
 <part name="SUPPLY5" library="supply2" deviceset="GND" device=""/>
 </parts>
@@
 <instance part="S5" gate="1" x="71.12" y="-5.08" rot="R270"/>
 <instance part="S2" gate="1" x="-68.58" y="83.82" rot="R270"/>
-<instance part="C8" gate="G$1" x="-68.58" y="-5.08"/>
+<instance part="C8" gate="G$1" x="-68.58" y="-2.54"/>
 <instance part="SUPPLY39" gate="GND" x="-68.58" y="-10.16"/>
 <instance part="C10" gate="G$1" x="-104.14" y="40.64" rot="R270"/>
-<instance part="GND2" gate="GND" x="-99.06" y="33.02"/>
+<instance part="GND2" gate="GND" x="-96.52" y="38.1"/>
 <instance part="C11" gate="G$1" x="-63.5" y="-81.28" rot="R270"/>
 <instance part="GND3" gate="GND" x="-50.8" y="-83.82"/>
@@
 <pinref part="C7" gate="G$1" pin="2"/>
 <pinref part="SUPPLY38" gate="GND" pin="GND"/>
-<wire x1="-134.62" y1="-12.7" x2="-134.62" y2="0" width="0.1524" layer="91"/>
+<wire x1="-134.62" y1="-12.7" x2="-134.62" y2="-2.54" width="0.1524" layer="91"/>
 </segment>
 <segment>
@@
 <segment>
 <pinref part="C10" gate="G$1" pin="1"/>
-<wire x1="-99.06" y1="40.64" x2="-99.06" y2="35.56" width="0.1524" layer="91"/>
+<wire x1="-101.6" y1="40.64" x2="-96.52" y2="40.64" width="0.1524" layer="91"/>
 <pinref part="GND2" gate="GND" pin="GND"/>
 </segment>
 <segment>
 <pinref part="C11" gate="G$1" pin="1"/>
-<wire x1="-58.42" y1="-81.28" x2="-50.8" y2="-81.28" width="0.1524" layer="91"/>
+<wire x1="-60.96" y1="-81.28" x2="-50.8" y2="-81.28" width="0.1524" layer="91"/>
 <pinref part="GND3" gate="GND" pin="GND"/>
 </segment>
@@
 <pinref part="C5" gate="G$1" pin="2"/>
 <pinref part="SUPPLY5" gate="GND" pin="GND"/>
+<wire x1="152.4" y1="55.88" x2="152.4" y2="53.34" width="0.1524" layer="91"/>
 </segment>
 </net>
@@
 <pinref part="FT232RL" gate="G$1" pin="DTR"/>
 <pinref part="C4" gate="G$1" pin="2"/>
-<wire x1="-78.74" y1="10.16" x2="-68.58" y2="10.16" width="0.1524" layer="91"/>
+<wire x1="-78.74" y1="10.16" x2="-71.12" y2="10.16" width="0.1524" layer="91"/>
 </segment>
 </net>
@@
 <pinref part="C4" gate="G$1" pin="1"/>
 <pinref part="ATMEGA" gate="G$1" pin="PC6(/RESET)"/>
-<wire x1="-48.26" y1="10.16" x2="-60.96" y2="10.16" width="0.1524" layer="91"/>
+<wire x1="-48.26" y1="10.16" x2="-63.5" y2="10.16" width="0.1524" layer="91"/>
 <junction x="-48.26" y="10.16"/>
 <wire x1="-48.26" y1="10.16" x2="-48.26" y2="17.78" width="0.1524" layer="91"/>
@@
 <junction x="-81.28" y="-81.28"/>
 <pinref part="C11" gate="G$1" pin="2"/>
-<wire x1="-71.12" y1="-81.28" x2="-66.04" y2="-81.28" width="0.1524" layer="91"/>
+<wire x1="-71.12" y1="-81.28" x2="-68.58" y2="-81.28" width="0.1524" layer="91"/>
 <junction x="-71.12" y="-81.28"/>
 </segment>
@@
 <wire x1="50.8" y1="73.66" x2="50.8" y2="68.58" width="0.1524" layer="91"/>
 <pinref part="R5" gate="G$1" pin="2"/>
-<wire x1="50.8" y1="68.58" x2="55.88" y2="68.58" width="0.1524" layer="91"/>
+<wire x1="50.8" y1="68.58" x2="60.96" y2="73.66" width="0.1524" layer="91"/>
 </segment>
 <segment>
@@
 <pinref part="U$3" gate="G$1" pin="VDD"/>
 <pinref part="P+20" gate="1" pin="+5V"/>
-<wire x1="127" y1="63.5" x2="152.4" y2="63.5" width="0.1524" layer="91"/>
-<wire x1="152.4" y1="63.5" x2="152.4" y2="66.04" width="0.1524" layer="91"/>
+<wire x1="127" y1="63.5" x2="152.4" y2="60.96" width="0.1524" layer="91"/>
+<wire x1="152.4" y1="60.96" x2="152.4" y2="66.04" width="0.1524" layer="91"/>
 <pinref part="C5" gate="G$1" pin="1"/>
-<junction x="152.4" y="63.5"/>
+<junction x="152.4" y="60.96"/>
 </segment>
 <segment>
@@
 <pinref part="C10" gate="G$1" pin="2"/>
 <wire x1="-111.76" y1="40.64" x2="-111.76" y2="50.8" width="0.1524" layer="91"/>
-<wire x1="-106.68" y1="40.64" x2="-111.76" y2="40.64" width="0.1524" layer="91"/>
+<wire x1="-109.22" y1="40.64" x2="-111.76" y2="40.64" width="0.1524" layer="91"/>
 <junction x="-111.76" y="40.64"/>
 </segment>
@@
 <wire x1="-109.22" y1="12.7" x2="-134.62" y2="12.7" width="0.1524" layer="91"/>
 <pinref part="C7" gate="G$1" pin="1"/>
-<wire x1="-134.62" y1="12.7" x2="-134.62" y2="7.62" width="0.1524" layer="91"/>
+<wire x1="-134.62" y1="12.7" x2="-134.62" y2="5.08" width="0.1524" layer="91"/>
 </segment>
 </net>
@@
 <pinref part="U$3" gate="G$1" pin="RST"/>
 <pinref part="R5" gate="G$1" pin="1"/>
-<wire x1="86.36" y1="68.58" x2="66.04" y2="68.58" width="0.1524" layer="91"/>
-</segment>
-</net>
+<wire x1="86.36" y1="68.58" x2="60.96" y2="66.04" width="0.1524" layer="91"/>
+</segment>
+</net>
