File: Stackduino-SMD.sch (EAGLE design)
At the start: 45 parts, among them CN1 Battery Connector, SW1 ROTARTY_ENCODER, Y1 16MHz

Commit message: latest progress
Parts:
- removed S5: (no value), adafruit:40-XX-ROUND
- added S1: (no value), adafruit:31-XX
- C1, C2, C3: device SparkFun-Capacitors:10NF-CER -> eagle-ltspice:CC1206
- S2: device adafruit:31-XX -> adafruit:40-XX-ROUND
- renumbered CN1 to BATT, JP1 to USB, JP2 to ICSP, OK1 to OPT2, OK3 to OPT1, SW1 to ROTARY_ENCODER, U$1 to DB15, U$3 to A4988_CARRIER
Connections:
- net GND: now also S1.P, S2.S1; no longer S2.P, S5.S1
- net N$28: now also S2.P1; no longer S5.P1
- net N$8: now also S1.S; no longer S2.S
Other:
- moved on the sheet: C1, C2, C3, C5, R5

Commit message: Latest progress
Connections:
- new net VIN: 12VDC.TIP, D2.A
- net V+: no longer 12VDC.TIP, D2.A
Other:
- moved on the sheet: D2
Changed lines of the file:
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@@
 <instance part="SUPPLY8" gate="GND" x="-99.06" y="63.5"/>
 <instance part="SUPPLY9" gate="GND" x="-152.4" y="96.52"/>
-<instance part="D2" gate="G$1" x="-111.76" y="127"/>
+<instance part="D2" gate="G$1" x="-109.22" y="127"/>
 <instance part="MP1" gate="G$1" x="-99.06" y="106.68" rot="R90"/>
 <instance part="SUPPLY12" gate="GND" x="-48.26" y="-48.26"/>
@@
 <junction x="-45.72" y="114.3"/>
 <pinref part="D2" gate="G$1" pin="C"/>
-<wire x1="-109.22" y1="127" x2="-68.58" y2="127" width="0.1524" layer="91"/>
+<wire x1="-106.68" y1="127" x2="-68.58" y2="127" width="0.1524" layer="91"/>
 <wire x1="-68.58" y1="127" x2="-68.58" y2="114.3" width="0.1524" layer="91"/>
 <junction x="-68.58" y="114.3"/>
@@
 <junction x="109.22" y="127"/>
 </segment>
-<segment>
-<pinref part="D2" gate="G$1" pin="A"/>
-<wire x1="-134.62" y1="127" x2="-114.3" y2="127" width="0.1524" layer="91"/>
-<pinref part="12VDC" gate="G$1" pin="TIP"/>
-<wire x1="-149.86" y1="134.62" x2="-134.62" y2="134.62" width="0.1524" layer="91"/>
-<wire x1="-134.62" y1="134.62" x2="-134.62" y2="127" width="0.1524" layer="91"/>
-<label x="-149.86" y="137.16" size="1.778" layer="95"/>
-</segment>
 </net>
 <net name="DIR" class="0">
@@
 </segment>
 </net>
+<net name="VIN" class="0">
+<segment>
+<pinref part="D2" gate="G$1" pin="A"/>
+<wire x1="-134.62" y1="127" x2="-111.76" y2="127" width="0.1524" layer="91"/>
+<pinref part="12VDC" gate="G$1" pin="TIP"/>
+<wire x1="-149.86" y1="134.62" x2="-134.62" y2="134.62" width="0.1524" layer="91"/>
+<wire x1="-134.62" y1="134.62" x2="-134.62" y2="127" width="0.1524" layer="91"/>
+<label x="-149.86" y="137.16" size="1.778" layer="95"/>
+</segment>
+</net>

Commit message: latest progress
Parts:
- removed C2: 68uF, eagle-ltspice:CC1206
- added C6: 68uF, SparkFun-Passives:CAP_POLD
- added L2: (no value), inductor-coilcraft:DO3316P
- C3: device eagle-ltspice:CC1206 -> SparkFun-Passives:CAP_POLD
- C9: value (none) -> 100uF
Connections:
- net GND: now also C3.-, C6.-; no longer C2.1, C3.1
- net V+: now also C3.+; no longer C3.2
- net VCC: now also C6.+; no longer C2.2
Other:
- moved on the sheet: C1
Changed lines of the file:
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@@
 <part name="C1" library="eagle-ltspice" deviceset="C" device="C1206" value="10nF"/>
 <part name="L1" library="SparkFun-Passives" deviceset="INDUCTOR" device="VLF4012A" value="47uH"/>
-<part name="C2" library="eagle-ltspice" deviceset="C" device="C1206" value="68uF"/>
-<part name="C3" library="eagle-ltspice" deviceset="C" device="C1206" value="100uF"/>
 <part name="SUPPLY1" library="supply2" deviceset="GND" device=""/>
-<part name="SUPPLY2" library="supply2" deviceset="GND" device=""/>
-<part name="SUPPLY3" library="supply2" deviceset="GND" device=""/>
 <part name="D1" library="SparkFun-DiscreteSemi" deviceset="MBRA140" device="" value="20v 1A"/>
 <part name="SUPPLY4" library="supply2" deviceset="GND" device=""/>
@@
 <part name="R19" library="rcl" deviceset="R-EU_" device="R1206" value="4.7K"/>
 <part name="P+17" library="supply1" deviceset="+5V" device="" value="VCC"/>
-<part name="C9" library="SparkFun-Passives" deviceset="CAP_POL" device="D"/>
+<part name="C9" library="SparkFun-Passives" deviceset="CAP_POL" device="D" value="100uF"/>
 <part name="S2" library="adafruit" deviceset="40-XX" device="-ROUND"/>
 <part name="S1" library="adafruit" deviceset="31-XX" device=""/>
@@
 <part name="C5" library="eagle-ltspice" deviceset="C" device="C1206" value="0.1uF"/>
 <part name="SUPPLY5" library="supply2" deviceset="GND" device=""/>
+<part name="C3" library="SparkFun-Passives" deviceset="CAP_POL" device="D" value="100uF"/>
+<part name="SUPPLY2" library="supply2" deviceset="GND" device=""/>
+<part name="C6" library="SparkFun-Passives" deviceset="CAP_POL" device="D" value="68uF"/>
+<part name="SUPPLY3" library="supply2" deviceset="GND" device=""/>
+<part name="L2" library="inductor-coilcraft" deviceset="DO3316P" device=""/>
 </parts>
 <sheets>
@@
 <instance part="LM2675" gate="A" x="12.7" y="109.22"/>
 <instance part="LTC4412" gate="A" x="-127" y="78.74" rot="R180"/>
-<instance part="C1" gate="G$1" x="38.1" y="109.22" rot="R90"/>
+<instance part="C1" gate="G$1" x="35.56" y="109.22" rot="R90"/>
 <instance part="L1" gate="G$1" x="48.26" y="104.14" rot="R90"/>
-<instance part="C2" gate="G$1" x="55.88" y="96.52" rot="R180"/>
-<instance part="C3" gate="G$1" x="-5.08" y="109.22" rot="R180"/>
 <instance part="SUPPLY1" gate="GND" x="2.54" y="83.82"/>
-<instance part="SUPPLY2" gate="GND" x="-5.08" y="93.98"/>
-<instance part="SUPPLY3" gate="GND" x="55.88" y="83.82"/>
 <instance part="D1" gate="G$1" x="40.64" y="91.44" rot="R90"/>
 <instance part="SUPPLY4" gate="GND" x="40.64" y="83.82"/>
@@
 <instance part="C5" gate="G$1" x="157.48" y="60.96"/>
 <instance part="SUPPLY5" gate="GND" x="157.48" y="50.8"/>
+<instance part="C3" gate="G$1" x="-7.62" y="106.68"/>
+<instance part="SUPPLY2" gate="GND" x="-7.62" y="99.06"/>
+<instance part="C6" gate="G$1" x="55.88" y="96.52"/>
+<instance part="SUPPLY3" gate="GND" x="55.88" y="86.36"/>
+<instance part="L2" gate="G$1" x="7.62" y="137.16"/>
 </instances>
 <busses>
@@
 <pinref part="LM2675" gate="A" pin="CB"/>
 <pinref part="C1" gate="G$1" pin="1"/>
-<wire x1="25.4" y1="109.22" x2="35.56" y2="109.22" width="0.1524" layer="91"/>
+<wire x1="25.4" y1="109.22" x2="33.02" y2="109.22" width="0.1524" layer="91"/>
 </segment>
 </net>
@@
 <wire x1="25.4" y1="104.14" x2="40.64" y2="104.14" width="0.1524" layer="91"/>
 <pinref part="C1" gate="G$1" pin="2"/>
-<wire x1="40.64" y1="104.14" x2="43.18" y2="109.22" width="0.1524" layer="91"/>
+<wire x1="40.64" y1="104.14" x2="40.64" y2="109.22" width="0.1524" layer="91"/>
 <pinref part="L1" gate="G$1" pin="1"/>
 <junction x="40.64" y="104.14"/>
@@
 <pinref part="LM2675" gate="A" pin="GND"/>
 <wire x1="2.54" y1="86.36" x2="2.54" y2="104.14" width="0.1524" layer="91"/>
-</segment>
-<segment>
-<pinref part="C3" gate="G$1" pin="1"/>
-<pinref part="SUPPLY2" gate="GND" pin="GND"/>
-<wire x1="-5.08" y1="96.52" x2="-5.08" y2="106.68" width="0.1524" layer="91"/>
-</segment>
-<segment>
-<pinref part="SUPPLY3" gate="GND" pin="GND"/>
-<pinref part="C2" gate="G$1" pin="1"/>
-<wire x1="55.88" y1="86.36" x2="55.88" y2="93.98" width="0.1524" layer="91"/>
 </segment>
 <segment>
@@
 <pinref part="SUPPLY5" gate="GND" pin="GND"/>
 <wire x1="157.48" y1="53.34" x2="157.48" y2="55.88" width="0.1524" layer="91"/>
+</segment>
+<segment>
+<pinref part="C3" gate="G$1" pin="-"/>
+<pinref part="SUPPLY2" gate="GND" pin="GND"/>
+</segment>
+<segment>
+<pinref part="C6" gate="G$1" pin="-"/>
+<pinref part="SUPPLY3" gate="GND" pin="GND"/>
+<wire x1="55.88" y1="88.9" x2="55.88" y2="91.44" width="0.1524" layer="91"/>
 </segment>
 </net>
@@
 </net>
 <net name="VCC" class="0">
-<segment>
-<pinref part="C2" gate="G$1" pin="2"/>
-<pinref part="L1" gate="G$1" pin="2"/>
-<wire x1="55.88" y1="101.6" x2="55.88" y2="104.14" width="0.1524" layer="91"/>
-<pinref part="LM2675" gate="A" pin="FB"/>
-<wire x1="25.4" y1="114.3" x2="25.4" y2="119.38" width="0.1524" layer="91"/>
-<wire x1="25.4" y1="119.38" x2="55.88" y2="119.38" width="0.1524" layer="91"/>
-<wire x1="55.88" y1="119.38" x2="55.88" y2="104.14" width="0.1524" layer="91"/>
-<junction x="55.88" y="104.14"/>
-<pinref part="P+2" gate="1" pin="+5V"/>
-<wire x1="55.88" y1="104.14" x2="68.58" y2="104.14" width="0.1524" layer="91"/>
-<wire x1="68.58" y1="104.14" x2="68.58" y2="106.68" width="0.1524" layer="91"/>
-</segment>
 <segment>
 <pinref part="R2" gate="G$1" pin="1"/>
@@
 <wire x1="-152.4" y1="86.36" x2="-152.4" y2="83.82" width="0.1524" layer="91"/>
 </segment>
+<segment>
+<pinref part="L1" gate="G$1" pin="2"/>
+<wire x1="55.88" y1="99.06" x2="55.88" y2="104.14" width="0.1524" layer="91"/>
+<pinref part="LM2675" gate="A" pin="FB"/>
+<wire x1="25.4" y1="114.3" x2="25.4" y2="119.38" width="0.1524" layer="91"/>
+<wire x1="25.4" y1="119.38" x2="55.88" y2="119.38" width="0.1524" layer="91"/>
+<wire x1="55.88" y1="119.38" x2="55.88" y2="104.14" width="0.1524" layer="91"/>
+<junction x="55.88" y="104.14"/>
+<pinref part="P+2" gate="1" pin="+5V"/>
+<wire x1="55.88" y1="104.14" x2="68.58" y2="104.14" width="0.1524" layer="91"/>
+<wire x1="68.58" y1="104.14" x2="68.58" y2="106.68" width="0.1524" layer="91"/>
+<pinref part="C6" gate="G$1" pin="+"/>
+</segment>
 </net>
 <net name="V+" class="0">
@@
 <wire x1="-109.22" y1="83.82" x2="-78.74" y2="83.82" width="0.1524" layer="91"/>
 <wire x1="-78.74" y1="83.82" x2="-78.74" y2="114.3" width="0.1524" layer="91"/>
-<pinref part="LM2675" gate="A" pin="VIN"/>
 <wire x1="-78.74" y1="114.3" x2="-68.58" y2="114.3" width="0.1524" layer="91"/>
-<pinref part="C3" gate="G$1" pin="2"/>
 <wire x1="-68.58" y1="114.3" x2="-45.72" y2="114.3" width="0.1524" layer="91"/>
 <wire x1="-45.72" y1="114.3" x2="-25.4" y2="114.3" width="0.1524" layer="91"/>
-<wire x1="-25.4" y1="114.3" x2="-5.08" y2="114.3" width="0.1524" layer="91"/>
-<wire x1="-5.08" y1="114.3" x2="2.54" y2="114.3" width="0.1524" layer="91"/>
-<junction x="-5.08" y="114.3"/>
 <pinref part="LTC2950" gate="A" pin="VIN"/>
 <wire x1="-45.72" y1="88.9" x2="-45.72" y2="114.3" width="0.1524" layer="91"/>
@@
 <junction x="-78.74" y="114.3"/>
 <wire x1="-25.4" y1="114.3" x2="-25.4" y2="127" width="0.1524" layer="91"/>
-<junction x="-25.4" y="114.3"/>
 <wire x1="-25.4" y1="127" x2="109.22" y2="127" width="0.1524" layer="91"/>
 <wire x1="109.22" y1="127" x2="109.22" y2="121.92" width="0.1524" layer="91"/>
@@
 <wire x1="127" y1="127" x2="127" y2="78.74" width="0.1524" layer="91"/>
 <junction x="109.22" y="127"/>
-</segment>
-</net>
+<wire x1="-25.4" y1="114.3" x2="-7.62" y2="114.3" width="0.1524" layer="91"/>
+<junction x="-25.4" y="114.3"/>
+<pinref part="LM2675" gate="A" pin="VIN"/>
+<pinref part="C3" gate="G$1" pin="+"/>
+<wire x1="-7.62" y1="114.3" x2="2.54" y2="114.3" width="0.1524" layer="91"/>
+<wire x1="-7.62" y1="109.22" x2="-7.62" y2="114.3" width="0.1524" layer="91"/>
+<junction x="-7.62" y="114.3"/>
+</segment>
+</net>

Commit message: Latest progress
Parts:
- removed L2: (no value), inductor-coilcraft:DO3316P
- removed Y1: 16MHz, SparkFun-FreqCtrl:RESONATOR16MHZ
- added C12, C2: (no value), eagle-ltspice:C
- added QF1: (no value), crystal:CRYSTALHC49U-V
- C1, C10, C11, C4, C5, C7, C8: device eagle-ltspice:CC1206 -> eagle-ltspice:C
- L1: device SparkFun-Passives:INDUCTORVLF4012A -> inductor-coilcraft:DO3316P
- R1, R18, R19, R2, R20, R21, R3, R4: device rcl:R-EU_R1206 -> eagle-ltspice:R
- R22: device eagle-ltspice:RR1206 -> eagle-ltspice:R
- R5: device eagle-ltspice:CC1206 -> eagle-ltspice:R
Connections:
- net GND: now also C12.2, C2.2; no longer Y1.2
- net N$15: now also C2.1, QF1.2; no longer Y1.3
- net N$16: now also C12.1, QF1.1; no longer Y1.1
Other:
- moved on the sheet: C1, C6, D1, R5

Commit message: latest progress
Parts:
- renumbered ATMEGA to ATMEGA328P
Connections:
- net N$25 renamed SCK
- net N$26 renamed MOSI
- net N$27 renamed MISO
Changed lines of the file:
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@@
 </classes>
 <parts>
-<part name="ATMEGA" library="SparkFun-DigitalIC" deviceset="ATMEGA328_SMT" device="" value="ATMEGA328P"/>
+<part name="ATMEGA328P" library="SparkFun-DigitalIC" deviceset="ATMEGA328_SMT" device="" value="ATMEGA328P"/>
 <part name="DB15" library="SparkFun-Connectors" deviceset="DB15" device=""/>
 <part name="ROTARY_ENCODER" library="SparkFun-Electromechanical" deviceset="ROTARTY_ENCODER" device=""/>
@@
 </plain>
 <instances>
-<instance part="ATMEGA" gate="G$1" x="-25.4" y="-15.24"/>
+<instance part="ATMEGA328P" gate="G$1" x="-25.4" y="-15.24"/>
 <instance part="DB15" gate="G$1" x="-198.12" y="35.56" rot="R90"/>
 <instance part="ROTARY_ENCODER" gate="G$1" x="-7.62" y="27.94"/>
@@
 </segment>
 <segment>
-<pinref part="ATMEGA" gate="G$1" pin="GND@2"/>
-<pinref part="ATMEGA" gate="G$1" pin="GND@1"/>
+<pinref part="ATMEGA328P" gate="G$1" pin="GND@2"/>
+<pinref part="ATMEGA328P" gate="G$1" pin="GND@1"/>
 <wire x1="-48.26" y1="-45.72" x2="-48.26" y2="-43.18" width="0.1524" layer="91"/>
-<pinref part="ATMEGA" gate="G$1" pin="AGND"/>
+<pinref part="ATMEGA328P" gate="G$1" pin="AGND"/>
 <wire x1="-48.26" y1="-40.64" x2="-48.26" y2="-43.18" width="0.1524" layer="91"/>
 <junction x="-48.26" y="-43.18"/>
@@
 <wire x1="-78.74" y1="48.26" x2="22.86" y2="48.26" width="0.1524" layer="91"/>
 <wire x1="22.86" y1="48.26" x2="22.86" y2="-15.24" width="0.1524" layer="91"/>
-<pinref part="ATMEGA" gate="G$1" pin="PD1(TXD)"/>
+<pinref part="ATMEGA328P" gate="G$1" pin="PD1(TXD)"/>
 <wire x1="22.86" y1="-15.24" x2="0" y2="-15.24" width="0.1524" layer="91"/>
 </segment>
@@
 <wire x1="-76.2" y1="45.72" x2="20.32" y2="45.72" width="0.1524" layer="91"/>
 <wire x1="20.32" y1="45.72" x2="20.32" y2="-12.7" width="0.1524" layer="91"/>
-<pinref part="ATMEGA" gate="G$1" pin="PD0(RXD)"/>
+<pinref part="ATMEGA328P" gate="G$1" pin="PD0(RXD)"/>
 <wire x1="20.32" y1="-12.7" x2="0" y2="-12.7" width="0.1524" layer="91"/>
 </segment>
@@
 <pinref part="R1" gate="G$1" pin="1"/>
 <pinref part="C4" gate="G$1" pin="1"/>
-<pinref part="ATMEGA" gate="G$1" pin="PC6(/RESET)"/>
+<pinref part="ATMEGA328P" gate="G$1" pin="PC6(/RESET)"/>
 <wire x1="-48.26" y1="10.16" x2="-63.5" y2="10.16" width="0.1524" layer="91"/>
 <junction x="-48.26" y="10.16"/>
@@
 <net name="N$15" class="0">
 <segment>
-<pinref part="ATMEGA" gate="G$1" pin="PB7(XTAL2/TOSC2)"/>
+<pinref part="ATMEGA328P" gate="G$1" pin="PB7(XTAL2/TOSC2)"/>
 <wire x1="-55.88" y1="-20.32" x2="-48.26" y2="-20.32" width="0.1524" layer="91"/>
 <pinref part="QF1" gate="G$1" pin="2"/>
@@
 <net name="N$16" class="0">
 <segment>
-<pinref part="ATMEGA" gate="G$1" pin="PB6(XTAL1/TOSC1)"/>
+<pinref part="ATMEGA328P" gate="G$1" pin="PB6(XTAL1/TOSC1)"/>
 <wire x1="-55.88" y1="-15.24" x2="-48.26" y2="-15.24" width="0.1524" layer="91"/>
 <pinref part="QF1" gate="G$1" pin="1"/>
@@
 <wire x1="-81.28" y1="-68.58" x2="63.5" y2="-68.58" width="0.1524" layer="91"/>
 <wire x1="63.5" y1="-68.58" x2="63.5" y2="-17.78" width="0.1524" layer="91"/>
-<pinref part="ATMEGA" gate="G$1" pin="PD2(INT0)"/>
+<pinref part="ATMEGA328P" gate="G$1" pin="PD2(INT0)"/>
 <wire x1="63.5" y1="-17.78" x2="0" y2="-17.78" width="0.1524" layer="91"/>
 </segment>
@@
 <wire x1="17.78" y1="-66.04" x2="58.42" y2="-66.04" width="0.1524" layer="91"/>
 <wire x1="58.42" y1="-66.04" x2="58.42" y2="-2.54" width="0.1524" layer="91"/>
-<pinref part="ATMEGA" gate="G$1" pin="PC5(ADC5/SCL)"/>
+<pinref part="ATMEGA328P" gate="G$1" pin="PC5(ADC5/SCL)"/>
 <wire x1="58.42" y1="-2.54" x2="0" y2="-2.54" width="0.1524" layer="91"/>
 <wire x1="17.78" y1="-66.04" x2="17.78" y2="-76.2" width="0.1524" layer="91"/>
@@
 <net name="N$19" class="0">
 <segment>
-<pinref part="ATMEGA" gate="G$1" pin="PC4(ADC4/SDA)"/>
+<pinref part="ATMEGA328P" gate="G$1" pin="PC4(ADC4/SDA)"/>
 <wire x1="0" y1="0" x2="53.34" y2="0" width="0.1524" layer="91"/>
 <wire x1="53.34" y1="0" x2="53.34" y2="-63.5" width="0.1524" layer="91"/>
@@
 <net name="N$22" class="0">
 <segment>
-<pinref part="ATMEGA" gate="G$1" pin="PB2(SS/OC1B)"/>
+<pinref part="ATMEGA328P" gate="G$1" pin="PB2(SS/OC1B)"/>
 <wire x1="0" y1="-40.64" x2="93.98" y2="-40.64" width="0.1524" layer="91"/>
 <wire x1="93.98" y1="-40.64" x2="93.98" y2="-58.42" width="0.1524" layer="91"/>
@@
 <net name="N$23" class="0">
 <segment>
-<pinref part="ATMEGA" gate="G$1" pin="PB0(ICP)"/>
+<pinref part="ATMEGA328P" gate="G$1" pin="PB0(ICP)"/>
 <wire x1="0" y1="-35.56" x2="83.82" y2="-35.56" width="0.1524" layer="91"/>
 <wire x1="83.82" y1="-35.56" x2="83.82" y2="-68.58" width="0.1524" layer="91"/>
@@
 <net name="N$24" class="0">
 <segment>
-<pinref part="ATMEGA" gate="G$1" pin="PB1(OC1A)"/>
+<pinref part="ATMEGA328P" gate="G$1" pin="PB1(OC1A)"/>
 <wire x1="0" y1="-38.1" x2="88.9" y2="-38.1" width="0.1524" layer="91"/>
 <wire x1="88.9" y1="-38.1" x2="88.9" y2="-63.5" width="0.1524" layer="91"/>
@@
 </segment>
 </net>
-<net name="N$25" class="0">
+<net name="SCK" class="0">
 <segment>
 <pinref part="ICSP" gate="G$1" pin="3"/>
@@
 <wire x1="129.54" y1="-27.94" x2="68.58" y2="-27.94" width="0.1524" layer="91"/>
 <wire x1="68.58" y1="-27.94" x2="68.58" y2="-48.26" width="0.1524" layer="91"/>
-<pinref part="ATMEGA" gate="G$1" pin="PB5(SCK)"/>
+<pinref part="ATMEGA328P" gate="G$1" pin="PB5(SCK)"/>
 <wire x1="68.58" y1="-48.26" x2="0" y2="-48.26" width="0.1524" layer="91"/>
 </segment>
 </net>
-<net name="N$26" class="0">
-<segment>
-<pinref part="ATMEGA" gate="G$1" pin="PB4(MISO)"/>
+<net name="MOSI" class="0">
+<segment>
+<pinref part="ATMEGA328P" gate="G$1" pin="PB4(MISO)"/>
 <wire x1="0" y1="-45.72" x2="73.66" y2="-45.72" width="0.1524" layer="91"/>
 <wire x1="73.66" y1="-45.72" x2="73.66" y2="-30.48" width="0.1524" layer="91"/>
@@
 </segment>
 </net>
-<net name="N$27" class="0">
-<segment>
-<pinref part="ATMEGA" gate="G$1" pin="PB3(MOSI/OC2)"/>
+<net name="MISO" class="0">
+<segment>
+<pinref part="ATMEGA328P" gate="G$1" pin="PB3(MOSI/OC2)"/>
 <wire x1="0" y1="-43.18" x2="78.74" y2="-43.18" width="0.1524" layer="91"/>
 <wire x1="78.74" y1="-43.18" x2="78.74" y2="-33.02" width="0.1524" layer="91"/>
@@
 <net name="N$28" class="0">
 <segment>
-<pinref part="ATMEGA" gate="G$1" pin="PD3(INT1)"/>
+<pinref part="ATMEGA328P" gate="G$1" pin="PD3(INT1)"/>
 <wire x1="0" y1="-20.32" x2="66.04" y2="-20.32" width="0.1524" layer="91"/>
 <wire x1="66.04" y1="-20.32" x2="66.04" y2="-7.62" width="0.1524" layer="91"/>
@@
 <net name="N$20" class="0">
 <segment>
-<pinref part="ATMEGA" gate="G$1" pin="PC0(ADC0)"/>
+<pinref part="ATMEGA328P" gate="G$1" pin="PC0(ADC0)"/>
 <wire x1="0" y1="10.16" x2="2.54" y2="10.16" width="0.1524" layer="91"/>
 <wire x1="2.54" y1="10.16" x2="2.54" y2="22.86" width="0.1524" layer="91"/>
@@
 <net name="N$21" class="0">
 <segment>
-<pinref part="ATMEGA" gate="G$1" pin="PC1(ADC1)"/>
+<pinref part="ATMEGA328P" gate="G$1" pin="PC1(ADC1)"/>
 <wire x1="0" y1="7.62" x2="5.08" y2="7.62" width="0.1524" layer="91"/>
 <wire x1="5.08" y1="7.62" x2="5.08" y2="33.02" width="0.1524" layer="91"/>
@@
 <net name="N$31" class="0">
 <segment>
-<pinref part="ATMEGA" gate="G$1" pin="PD6(AIN0)"/>
+<pinref part="ATMEGA328P" gate="G$1" pin="PD6(AIN0)"/>
 <wire x1="0" y1="-27.94" x2="40.64" y2="-27.94" width="0.1524" layer="91"/>
 <wire x1="40.64" y1="-27.94" x2="40.64" y2="40.64" width="0.1524" layer="91"/>
@@
 <net name="N$32" class="0">
 <segment>
-<pinref part="ATMEGA" gate="G$1" pin="PD7(AIN1)"/>
+<pinref part="ATMEGA328P" gate="G$1" pin="PD7(AIN1)"/>
 <wire x1="0" y1="-30.48" x2="43.18" y2="-30.48" width="0.1524" layer="91"/>
 <wire x1="43.18" y1="-30.48" x2="43.18" y2="20.32" width="0.1524" layer="91"/>
@@
 <net name="ALOG1" class="0">
 <segment>
-<pinref part="ATMEGA" gate="G$1" pin="PC2(ADC2)"/>
+<pinref part="ATMEGA328P" gate="G$1" pin="PC2(ADC2)"/>
 <wire x1="0" y1="5.08" x2="5.08" y2="5.08" width="0.1524" layer="91"/>
 <label x="7.62" y="5.08" size="1.778" layer="95"/>
@@
 <net name="ALOG2" class="0">
 <segment>
-<pinref part="ATMEGA" gate="G$1" pin="PC3(ADC3)"/>
+<pinref part="ATMEGA328P" gate="G$1" pin="PC3(ADC3)"/>
 <wire x1="0" y1="2.54" x2="5.08" y2="2.54" width="0.1524" layer="91"/>
 <label x="7.62" y="2.54" size="1.778" layer="95"/>
@@
 </segment>
 <segment>
-<pinref part="ATMEGA" gate="G$1" pin="AREF"/>
-<pinref part="ATMEGA" gate="G$1" pin="VCC@2"/>
+<pinref part="ATMEGA328P" gate="G$1" pin="AREF"/>
+<pinref part="ATMEGA328P" gate="G$1" pin="VCC@2"/>
 <wire x1="-48.26" y1="-5.08" x2="-48.26" y2="0" width="0.1524" layer="91"/>
-<pinref part="ATMEGA" gate="G$1" pin="VCC@1"/>
+<pinref part="ATMEGA328P" gate="G$1" pin="VCC@1"/>
 <wire x1="-48.26" y1="0" x2="-48.26" y2="2.54" width="0.1524" layer="91"/>
 <junction x="-48.26" y="0"/>
-<pinref part="ATMEGA" gate="G$1" pin="AVCC"/>
+<pinref part="ATMEGA328P" gate="G$1" pin="AVCC"/>
 <wire x1="-48.26" y1="2.54" x2="-48.26" y2="5.08" width="0.1524" layer="91"/>
 <junction x="-48.26" y="2.54"/>
@@
 <net name="DIR" class="0">
 <segment>
-<pinref part="ATMEGA" gate="G$1" pin="PD4(XCK/T0)"/>
+<pinref part="ATMEGA328P" gate="G$1" pin="PD4(XCK/T0)"/>
 <wire x1="0" y1="-22.86" x2="30.48" y2="-22.86" width="0.1524" layer="91"/>
 <wire x1="30.48" y1="-22.86" x2="30.48" y2="60.96" width="0.1524" layer="91"/>
@@
 <net name="STEP" class="0">
 <segment>
-<pinref part="ATMEGA" gate="G$1" pin="PD5(T1)"/>
+<pinref part="ATMEGA328P" gate="G$1" pin="PD5(T1)"/>
 <wire x1="0" y1="-25.4" x2="33.02" y2="-25.4" width="0.1524" layer="91"/>
 <wire x1="33.02" y1="-25.4" x2="33.02" y2="63.5" width="0.1524" layer="91"/>
