File: Stackduino-SMD.sch (EAGLE design)
At the start: 47 parts

Commit message: Latest progress
Parts:
- added C13: 22uF, eagle-ltspice:C
- added R6: 10K, eagle-ltspice:R
- MP1: value (none) -> FDN306P
Connections:
- net GND: now also C13.2
- net KILL: now also R6.1
- net V+: now also C13.1
- net VCC: now also R6.2
Changed lines of the file:
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@@
 <part name="SUPPLY9" library="supply2" deviceset="GND" device=""/>
 <part name="D2" library="SparkFun-DiscreteSemi" deviceset="MBRA140" device="" value="20v 1A"/>
-<part name="MP1" library="sym" deviceset="PMOS" device=""/>
+<part name="MP1" library="sym" deviceset="PMOS" device="" value="FDN306P"/>
 <part name="SUPPLY12" library="supply2" deviceset="GND" device=""/>
 <part name="SUPPLY14" library="supply2" deviceset="GND" device=""/>
@@
 <part name="SUPPLY6" library="supply2" deviceset="GND" device=""/>
 <part name="SUPPLY11" library="supply2" deviceset="GND" device=""/>
+<part name="C13" library="eagle-ltspice" deviceset="C" device="" value="22uF"/>
+<part name="GND4" library="supply2" deviceset="GND" device=""/>
+<part name="R6" library="eagle-ltspice" deviceset="R" device="" value="10K"/>
+<part name="P+3" library="supply1" deviceset="+5V" device="" value="VCC"/>
 </parts>
 <sheets>
@@
 <instance part="D1" gate="G$1" x="43.18" y="93.98" rot="R90"/>
 <instance part="SUPPLY4" gate="GND" x="43.18" y="86.36"/>
-<instance part="GND" gate="GND" x="-73.66" y="63.5"/>
+<instance part="GND" gate="GND" x="-73.66" y="73.66"/>
 <instance part="SUPPLY7" gate="GND" x="-45.72" y="63.5"/>
 <instance part="SUPPLY8" gate="GND" x="-99.06" y="63.5"/>
@@
 <instance part="SUPPLY6" gate="GND" x="-63.5" y="-33.02"/>
 <instance part="SUPPLY11" gate="GND" x="-73.66" y="-33.02"/>
+<instance part="C13" gate="G$1" x="-60.96" y="104.14"/>
+<instance part="GND4" gate="GND" x="-60.96" y="96.52"/>
+<instance part="R6" gate="G$1" x="-66.04" y="63.5" rot="R180"/>
+<instance part="P+3" gate="1" x="-86.36" y="66.04" smashed="yes">
+<attribute name="VALUE" x="-84.074" y="64.262" size="1.778" layer="96"/>
+</instance>
 </instances>
 <busses>
@@
 </segment>
 <segment>
-<wire x1="-73.66" y1="83.82" x2="-73.66" y2="66.04" width="0.1524" layer="91"/>
+<wire x1="-73.66" y1="83.82" x2="-73.66" y2="76.2" width="0.1524" layer="91"/>
 <pinref part="GND" gate="GND" pin="GND"/>
 <pinref part="S1" gate="1" pin="P"/>
@@
 <pinref part="SUPPLY11" gate="GND" pin="GND"/>
 <wire x1="-73.66" y1="-30.48" x2="-73.66" y2="-33.02" width="0.1524" layer="91"/>
+</segment>
+<segment>
+<pinref part="C13" gate="G$1" pin="2"/>
+<pinref part="GND4" gate="GND" pin="GND"/>
 </segment>
 </net>
@@
 <pinref part="LTC2950" gate="A" pin="~KILL"/>
 <wire x1="-45.72" y1="78.74" x2="-60.96" y2="78.74" width="0.1524" layer="91"/>
-<wire x1="-60.96" y1="78.74" x2="-60.96" y2="58.42" width="0.1524" layer="91"/>
+<wire x1="-60.96" y1="78.74" x2="-60.96" y2="63.5" width="0.1524" layer="91"/>
 <label x="-63.5" y="55.88" size="1.778" layer="95"/>
+<pinref part="R6" gate="G$1" pin="1"/>
+<wire x1="-60.96" y1="63.5" x2="-60.96" y2="58.42" width="0.1524" layer="91"/>
+<junction x="-60.96" y="63.5"/>
 </segment>
 <segment>
@@
 <pinref part="C6" gate="G$1" pin="+"/>
 </segment>
+<segment>
+<pinref part="R6" gate="G$1" pin="2"/>
+<wire x1="-71.12" y1="63.5" x2="-86.36" y2="63.5" width="0.1524" layer="91"/>
+<pinref part="P+3" gate="1" pin="+5V"/>
+</segment>
 </net>
 <net name="V+" class="0">
@@
 <wire x1="-78.74" y1="83.82" x2="-78.74" y2="114.3" width="0.1524" layer="91"/>
 <wire x1="-78.74" y1="114.3" x2="-68.58" y2="114.3" width="0.1524" layer="91"/>
-<wire x1="-68.58" y1="114.3" x2="-45.72" y2="114.3" width="0.1524" layer="91"/>
+<wire x1="-68.58" y1="114.3" x2="-60.96" y2="114.3" width="0.1524" layer="91"/>
+<wire x1="-60.96" y1="114.3" x2="-45.72" y2="114.3" width="0.1524" layer="91"/>
 <wire x1="-45.72" y1="114.3" x2="-25.4" y2="114.3" width="0.1524" layer="91"/>
 <pinref part="LTC2950" gate="A" pin="VIN"/>
@@
 <wire x1="-7.62" y1="109.22" x2="-7.62" y2="114.3" width="0.1524" layer="91"/>
 <junction x="-7.62" y="114.3"/>
-</segment>
-</net>
+<pinref part="C13" gate="G$1" pin="1"/>
+<wire x1="-60.96" y1="106.68" x2="-60.96" y2="114.3" width="0.1524" layer="91"/>
+<junction x="-60.96" y="114.3"/>
+</segment>
+</net>

Commit message: latest progress
Parts:
- removed R18, R19: 4.7K, eagle-ltspice:R
- removed R22: 470K, eagle-ltspice:R
- added R10: 1.5K, eagle-ltspice:R
- added R7: 220K, eagle-ltspice:R
- C1: value 10nF -> 22uF
- C10: value 0.1uF -> 100nF
- C11: value 0.1uF -> (none)
- C13: value 22uF -> 0.1uF
- C2: value (none) -> 100uF; device eagle-ltspice:C -> SparkFun-Passives:CAP_POLD
- C3: value 100uF -> 10nF; device SparkFun-Passives:CAP_POLD -> eagle-ltspice:C
- C4: value 0.1uF -> 68uF; device eagle-ltspice:C -> SparkFun-Passives:CAP_POLD
- C6: value 68uF -> 100uF
- C7: value 100nF -> 0.1uF
- C9: value 100uF -> 0.1uF; device SparkFun-Passives:CAP_POLD -> eagle-ltspice:C
- R1: value 1.5K -> 470K
- R3, R4: value 220K -> 4.7K
- R6: value 10K -> 220K
- renumbered R20 to R9, R21 to R8
Connections:
- net GND: now also C1.2, C10.2, C11.2, C2.-, C4.-, C5.1, C9.1, D2.A; no longer C10.1, C11.1, C2.2, C3.-, C5.2, C8.2, C9.-, D1.A
- net KILL: no longer R6.1
- net N$11: now also C8.1, R10.1; no longer C4.1, R1.1
- net N$15: now also C12.1; no longer C2.1
- net N$16: now also C11.1; no longer C12.1
- net N$18: now also R4.1; no longer R19.1
- net N$19: now also R3.2; no longer R18.2
- net N$3: now also C8.2; no longer C4.2
- net N$31: now also R6.2; no longer R3.2
- net N$32: now also R7.2; no longer R4.2
- net N$34: now also R6.1; no longer R3.1
- net N$36: now also R7.1; no longer R4.1
- net N$4: now also C3.1; no longer C1.1
- net N$43: now also C10.1; no longer C7.1
- net N$7: now also C3.2, D2.C; no longer C1.2, D1.C
- net STAT: now also R1.1; no longer R22.1
- net V+: now also C1.1, C2.+, C6.+, D1.C; no longer C13.1, C3.+, C9.+, D2.C
- net VCC: now also C13.1, C4.+, C5.2, C7.1, C9.2, R10.2, R3.1, R4.2; no longer C10.2, C11.2, C5.1, C6.+, C8.1, R18.1, R19.2, R22.2, R6.2
- net VIN: now also D1.A; no longer D2.A
Other:
- moved on the sheet: C1, C10, C11, C12, C13, C5, C6, C7, C8, D1, D2, R1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

Commit message: latest progress
Parts:
- removed ROTARY_ENCODER: ROTARTY_ENCODER, SparkFun-Electromechanical:ROTARTY_ENCODER
- removed S1: (no value), adafruit:31-XX
- removed S2: (no value), adafruit:40-XX-ROUND
- removed S3: Forward, SparkFun-Electromechanical:TAC_SWITCHPTH
- removed S4: Backward, SparkFun-Electromechanical:TAC_SWITCHPTH
- added ENCODER: JST-PH_3-PIN_HEADER, SRG:JST-PH_3-PIN_HEADER
- added FWD/BWD: JST-PH_4-PIN_HEADER, SRG:JST-PH_4-PIN_HEADER
- added MENU_SEL, ON/OFF, START/STOP: JST-PH_2-PIN_HEADER, SRG:JST-PH_2-PIN_HEADER
- BATT: device adafruit:JST_2PIN-THM -> adafruit:JST_2PIN-THM-RA
Connections:
- net N$15 renamed XTAL2
- net N$16 renamed XTAL1
- net N$31 renamed PD6
- net N$32 renamed PD7
- removed net N$20: ATMEGA328P.PC0(ADC0), ROTARY_ENCODER.A
- removed net N$21: ATMEGA328P.PC1(ADC1), ROTARY_ENCODER.B
- new net PC0: ATMEGA328P.PC0(ADC0), ENCODER.1
- new net PC1: ATMEGA328P.PC1(ADC1), ENCODER.3
- net ENCSWITCH: now also MENU_SEL.2; no longer ROTARY_ENCODER.SW-
- net GND: now also ENCODER.2, FWD/BWD.1, FWD/BWD.3, MENU_SEL.1, ON/OFF.2, START/STOP.1; no longer ROTARY_ENCODER.C, ROTARY_ENCODER.SW+, S1.P, S2.S1, S3.2, S4.2
- net MISO: now also ATMEGA328P.PB4(MISO); no longer ATMEGA328P.PB3(MOSI/OC2)
- net MOSI: now also ATMEGA328P.PB3(MOSI/OC2); no longer ATMEGA328P.PB4(MISO)
- net N$28: now also START/STOP.2; no longer S2.P1
- net N$33: now also FWD/BWD.2; no longer S4.4
- net N$35: now also FWD/BWD.4; no longer S3.4
- net N$8: now also ON/OFF.1; no longer S1.S
